File: Hardware/TheAaahhhDeviceHW/TheAaahhhDeviceHW.kicad_pcb (KiCad board)
At the start: 2 copper layers, 9 parts, among them J1 Speaker, J2 WS_LEDStrip, U1 WeMos_D1_mini, U2 DFPlayerMini

Commit message: 2022-10-23
Parts:
- added C1: 100n, Capacitor_SMD:C_0805_2012Metric_Pad1.18x1.45mm_HandSolder, F.Cu at (132.3, 152.7)
- added C2: 100n, Capacitor_SMD:C_0805_2012Metric_Pad1.18x1.45mm_HandSolder, F.Cu at (119.6, 152.7)
- added J3: WeMos_D1_Breakout, Connector_PinHeader_2.54mm:PinHeader_1x08_P2.54mm_Vertical, F.Cu at (147.8, 93.1)
- added J4: DFPlayerMini_Breakout, Connector_PinHeader_2.54mm:PinHeader_1x08_P2.54mm_Vertical, F.Cu at (144.9, 124.7)
- moved R3 9.65 mm to (136.4, 124.5)
- moved J2 0.76 mm to (128.3, 158.2)
Connections:
- U1 pad 1: unconnected-(U1-Pad1) -> RST
- U1 pad 11: unconnected-(U1-Pad11) -> D4
- U1 pad 12: unconnected-(U1-Pad12) -> D3
- U1 pad 13: unconnected-(U1-Pad13) -> D2
- U1 pad 14: unconnected-(U1-Pad14) -> D1
- U1 pad 15: unconnected-(U1-Pad15) -> RX
- U1 pad 16: unconnected-(U1-Pad16) -> TX
- U1 pad 3: unconnected-(U1-Pad3) -> D0
- U2 pad 11: unconnected-(U2-Pad11) -> DF_IO2
- U2 pad 12: unconnected-(U2-Pad12) -> DF_ADKEY1
- U2 pad 13: unconnected-(U2-Pad13) -> DF_ADKEY2
- U2 pad 14: unconnected-(U2-Pad14) -> DF_USB+
- U2 pad 15: unconnected-(U2-Pad15) -> DF_USB-
- U2 pad 4: unconnected-(U2-Pad4) -> DF_DAC_R
- U2 pad 5: unconnected-(U2-Pad5) -> DF_DAC_L
- U2 pad 9: unconnected-(U2-Pad9) -> DF_IO1
Routing:
- net +5V: track 0.00 -> 90.3 mm
- net WS_DIn: track 0.00 -> 52.8 mm
- net DF_Busy: track 0.00 -> 42.9 mm
- net DF_DAC_L: track 0.00 -> 35.4 mm
- net D0: track 0.00 -> 32.6 mm
- net +3V3: track 0.00 -> 31.3 mm
- net RST: track 0.00 -> 29.8 mm
- net DF_TX: track 0.00 -> 29.8 mm
- net TX: track 0.00 -> 28.1 mm
- net DF_RX: track 0.00 -> 27.8 mm
- net DF_DAC_R: track 0.00 -> 26.3 mm
- net RX: track 0.00 -> 25.5 mm
- net WS_DOut: track 0.00 -> 25.0 mm, vias 0 -> 1
- net DF_IO2: track 0.00 -> 12.7 mm
- net DF_ADKEY2: track 0.00 -> 12.6 mm
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- added copper zone on B.Cu, net GND
- added copper zone on F.Cu, net GND
Other:
- board text added: "ADKey 1"
- board text added: "ADKey 2"
- board text added: "D0"
- board text added: "D1"
- board text added: "D2"
- board text added: "D3"
- board text added: "D4"
- board text added: "DAC_L"
- board text added: "DAC_R"
- board text added: "DFPlayer Mini:"
- board text added: "IO 1"
- board text added: "IO 2"
- board text added: "RST"
- board text added: "RX"
- board text added: "TX"
- board text added: "USB+"
- board text added: "USB-"
- board text added: "WeMos:"

Commit message: 2022-10-24
Other:
- board text added: "Aaahhh"
- board text added: "Call286"
Changed lines of the file:
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@@
     (effects (font (size 1.5 1.5) (thickness 0.3)))
+  )
+  (gr_text "Aaahhh" (at 152.4 154.94) (layer "F.SilkS")
+    (effects (font (size 3 3) (thickness 0.5)))
   )
   (gr_text "IO 1" (at 150.114 140.208) (layer "F.SilkS")
@@
     (effects (font (size 1.5 1.5) (thickness 0.3)))
   )
+  (gr_text "Call286" (at 152.4 158.75) (layer "F.SilkS")
+    (effects (font (size 1.5 1.5) (thickness 0.3)))
+  )
