File: Hardware/TheAaahhhDeviceHW/TheAaahhhDeviceHW.kicad_sch (KiCad schematic)
At the start: 6 parts

Commit message: 2022-10-17
Parts:
- added D1, D2: WS2812, LED_SMD:LED_WS2812_PLCC6_5.0x5.0mm_P1.6mm, symbol LED:WS2812
- added J1: Speaker, Connector_PinHeader_2.54mm:PinHeader_1x02_P2.54mm_Vertical, symbol Connector:Conn_01x02_Male
- J2: renamed from J?; value NeoPixel -> WS_LEDStrip; footprint (none) -> Connector_PinHeader_2.54mm:PinHeader_1x03_P2.54mm_Vertical
- R1: renamed from R?; footprint (none) -> OptoDevice:R_LDR_5.1x4.3mm_P3.4mm_Vertical
- R2, R3: renamed from R?; footprint (none) -> Resistor_THT:R_Axial_DIN0207_L6.3mm_D2.5mm_P10.16mm_Horizontal
- gave numbers to parts that had none: 2
Connections:
- net +5V: now also U1.9 (5V), U2.1 (VCC), D1.3 (VCC), D1.5 (VDD), D2.3 (VCC), D2.5 (VDD)
- net GND: now also R2.2, R3.2, U1.10 (GND), U2.10 (GND), U2.7 (GND), D1.6 (VSS), D2.6 (VSS)
- net DF_Busy: now reaches U2.16 (BUSY)
- net DF_Busy: now also R3.1, U1.4 (SCK/D5)
- net DF_RX: now reaches U2.2 (RX)
- net DF_RX: now also U1.5 (MISO/D6)
- net DF_TX: now reaches U2.3 (TX)
- net DF_TX: now also U1.6 (MOSI/D7)
- net DF_SPK1: now reaches U2.6 (SPK1)
- net DF_SPK1: now also J1.2 (Pin_2)
- net DF_SPK2: now reaches U2.8 (SPK2)
- net DF_SPK2: now also J1.1 (Pin_1)
- net +3V3: now reaches R1.1
- net +3V3: now also U1.8 (3V3)
- net A0: now reaches R1.2
- net A0: now also R2.1, U1.2 (A0)
- net WS_DIn: now reaches U1.7 (CS/D8)
- net WS_DIn: now also D1.2 (DIN)
- net DI renamed WS_DOut
- net WS_DOut: now also D1.1 (DOUT), D2.2 (DIN)
- no-connect marks 0 -> 17
Other:
- moved on the sheet: J2, R1, R2, R3, U2

Commit message: 2022-10-23
Parts:
- added C1, C2: 100n, Capacitor_SMD:C_0805_2012Metric_Pad1.18x1.45mm_HandSolder, symbol Device:C
- added J3: WeMos_D1_Breakout, Connector_PinHeader_2.54mm:PinHeader_1x08_P2.54mm_Vertical, symbol Connector:Conn_01x08_Male
- added J4: DFPlayerMini_Breakout, Connector_PinHeader_2.54mm:PinHeader_1x08_P2.54mm_Vertical, symbol Connector:Conn_01x08_Male
Connections:
- net +5V: now also C1.2, C2.2
- net GND: now also C1.1, C2.1
- net DF_IO2: now reaches U2.11 (IO2)
- net DF_IO2: now also J4.8 (Pin_8)
- net DF_ADKEY1: now reaches U2.12 (ADKEY1)
- net DF_ADKEY1: now also J4.5 (Pin_5)
- net DF_ADKEY2: now reaches U2.13 (ADKEY2)
- net DF_ADKEY2: now also J4.6 (Pin_6)
- net DF_USB+: now reaches U2.14 (USB+)
- net DF_USB+: now also J4.4 (Pin_4)
- net DF_USB-: now reaches U2.15 (USB-)
- net DF_USB-: now also J4.3 (Pin_3)
- net DF_DAC_R: now reaches U2.4 (DAC_R)
- net DF_DAC_R: now also J4.2 (Pin_2)
- net DF_DAC_L: now reaches U2.5 (DAC_L)
- net DF_DAC_L: now also J4.1 (Pin_1)
- net DF_IO1: now reaches U2.9 (IO1)
- net DF_IO1: now also J4.7 (Pin_7)
- net RST: now reaches U1.1 (~{RST})
- net RST: now also J3.1 (Pin_1)
- net D4: now reaches U1.11 (D4)
- net D4: now also J3.6 (Pin_6)
- net D3: now reaches U1.12 (D3)
- net D3: now also J3.5 (Pin_5)
- net D2: now reaches U1.13 (SDA/D2)
- net D2: now also J3.4 (Pin_4)
- net D1: now reaches U1.14 (SCL/D1)
- net D1: now also J3.3 (Pin_3)
- net RX: now reaches U1.15 (RX)
- net RX: now also J3.8 (Pin_8)
- net TX: now reaches U1.16 (TX)
- net TX: now also J3.7 (Pin_7)
- net D0: now reaches U1.3 (D0)
- net D0: now also J3.2 (Pin_2)
- no-connect marks 17 -> 1

Commit message: v1
Parts:
- added H1, H2, H3, H4: MountingHole, MountingHole:MountingHole_3.2mm_M3_Pad_Via, symbol Mechanical:MountingHole_Pad
- added JP1: Bridge_DIN_To_DOUT, Jumper:SolderJumper-2_P1.3mm_Open_RoundedPad1.0x1.5mm, symbol Jumper:Jumper_2_Open
- D1, D2: footprint LED_SMD:LED_WS2812_PLCC6_5.0x5.0mm_P1.6mm -> DCDModules:LED_WS2812+SMD
Connections:
- net GND: now also H1.1, H2.1, H3.1, H4.1
- net WS_DIn: now also JP1.1 (A)
- net WS_DOut: no longer J2.2 (Pin_2)
- new net WS_DInOut: J2.2 (Pin_2), JP1.2 (B)
